File: mcu.kicad_sch (KiCad schematic)
At the start: 3 parts, among them SW1 RotaryEncoder_Switch, SW2 RotaryEncoder_Switch, U2 BluePill

Commit message: Progress.
Connections:
- net +VBUS: now reaches U2.18 (5V)
- net GND: now reaches U2.19 (GND)
- net GND: now also U2.39 (GND), U2.40 (GND), U2.41 (GND)
- net SQUARE_SEL: now reaches U2.26 (PA1)
- net PWM_SEL: now reaches U2.27 (PA2)
- net DC_OFFSET_PWM: now reaches U2.28 (PA3)
- net PWM_THRS_DAC: now reaches U2.29 (PA4)

Commit message: Savegame.
Parts:
- removed SW1, SW2: RotaryEncoder_Switch, Rotary_Encoder:RotaryEncoder_Bourns_Vertical_PEC12R-3x17F-Sxxxx, symbol Device:RotaryEncoder_Switch
- added C45, C46, C47, C48, C49, C50: 10n, Resistor_SMD:R_0603_1608Metric_Pad0.98x0.95mm_HandSolder, symbol Device:C
- added J3: Conn_01x02_Pin, Connector_PinHeader_2.54mm:PinHeader_1x02_P2.54mm_Vertical, symbol Connector:Conn_01x02_Pin
- added J5: Conn_01x04_Pin, Connector_PinHeader_2.54mm:PinHeader_1x04_P2.54mm_Vertical, symbol Connector:Conn_01x04_Pin
- added R36, R37, R38, R39, R40, R41, R42, R43, R44, R45, R46, R47: 10k, Resistor_SMD:R_0603_1608Metric_Pad0.98x0.95mm_HandSolder, symbol Device:R_US
- added SW1, SW2: RotaryEncoder_Switch, PSG:RotaryEncoder_Bourns_Vertical_PEC12R-3x17F-Sxxxx, symbol PSG:RotaryEncoder_Switch
- added U16: Screen to I2C, PSG:screen_to_i2c, symbol PSG:Screen_to_I2C
- added U17: Screen, PSG:20x4 screen, symbol PSG:20x4_screen
Connections:
- net +VBUS: now also J5.2 (Pin_2)
- net DC_OFFSET_PWM: now also U2.26 (PA1); no longer U2.28 (PA3)
- net GND: now also C45.1, C46.1, C47.1, C48.1, C49.1, C50.1, J5.1 (Pin_1), SW1.C, SW1.S2, SW2.C, SW2.S2
- net PWM_SEL: now also U2.23 (PC14); no longer U2.27 (PA2)
- net PWM_THRS_DAC: now also U2.27 (PA2); no longer U2.29 (PA4)
- net SQUARE_SEL: now also U2.22 (PC13); no longer U2.26 (PA1)
- net EN_A_2: now reaches U2.1 (PB12)
- net EN_A_2: now also C48.2, R43.1
- net SCL_1: now reaches U2.14 (PB6)
- net SCL_1: now also J5.4 (Pin_4)
- net SDA_1: now reaches U2.15 (PB7)
- net SDA_1: now also J5.3 (Pin_3)
- net SDA_2: now reaches U2.16 (PB8)
- net SCL_2: now reaches U2.17 (PB9)
- net EN_B_2: now reaches U2.2 (PB13)
- net EN_B_2: now also C49.2, R45.1
- net +3.3V_MCU: now reaches U2.20 (3V3)
- net +3.3V_MCU: now also U2.38 (3V3), U2.44 (3V3), J3.2 (Pin_2)
- net EN_SW_2: now reaches U2.3 (PB14)
- net EN_SW_2: now also C50.2, R47.1
- net SCK_SG: now reaches U2.30 (PA5)
- net SDATA_SG: now reaches U2.32 (PA7)
- net FSYNC_SG: now reaches U2.33 (PB0)
- net EN_A_1: now reaches U2.4 (PB15)
- net EN_A_1: now also C45.2, R39.1
- net EN_B_1: now reaches U2.5 (PA8)
- net EN_B_1: now also C46.2, R37.1
- net EN_SW_1: now reaches U2.6 (PA9)
- net EN_SW_1: now also C47.2, R41.1
- new net: R38.1, R39.2, SW1.A
- new net: R44.1, R45.2, SW2.B
- new net: R40.1, R41.2, SW1.S1
- new net: R42.1, R43.2, SW2.A
- new net: R46.1, R47.2, SW2.S1
- new net: R36.1, R37.2, SW1.B
- new net +3.3V: J3.1 (Pin_1), R36.2, R38.2, R40.2, R42.2, R44.2, R46.2
Other:
- note added: "3V3 source sel"
- note added: "Menu encoder"
- note added: "Screen I2C"
- note added: "Value encoder"
