File: PSG10M.kicad_pcb (KiCad board)
At the start: 2 copper layers, 3 parts, among them SW1 RotaryEncoder_Switch, U1 AD8933_module, U2 BluePill

Commit message: Ide nekako idk.
Parts:
- added R1: 1k, Resistor_SMD:R_0603_1608Metric_Pad0.98x0.95mm_HandSolder, F.Cu at (129.9, 121.0)
- added R10: 100k, Resistor_SMD:R_0603_1608Metric_Pad0.98x0.95mm_HandSolder, F.Cu at (138.6, 123.5)
- added R11: 1k, Resistor_SMD:R_0603_1608Metric_Pad0.98x0.95mm_HandSolder, F.Cu at (138.6, 126.0)
- added R12: 2k, Resistor_SMD:R_0603_1608Metric_Pad0.98x0.95mm_HandSolder, F.Cu at (138.6, 128.5)
- added R2: 2k, Resistor_SMD:R_0603_1608Metric_Pad0.98x0.95mm_HandSolder, F.Cu at (129.9, 123.5)
- added R3: 1k, Resistor_SMD:R_0603_1608Metric_Pad0.98x0.95mm_HandSolder, F.Cu at (129.9, 126.0)
- added R4: 2k, Resistor_SMD:R_0603_1608Metric_Pad0.98x0.95mm_HandSolder, F.Cu at (129.9, 128.5)
- added R5: 100k, Resistor_SMD:R_0603_1608Metric_Pad0.98x0.95mm_HandSolder, F.Cu at (134.3, 121.0)
- added R6: 100k, Resistor_SMD:R_0603_1608Metric_Pad0.98x0.95mm_HandSolder, F.Cu at (134.3, 123.5)
- added R7: 1k, Resistor_SMD:R_0603_1608Metric_Pad0.98x0.95mm_HandSolder, F.Cu at (134.3, 126.0)
- added R8: 2k, Resistor_SMD:R_0603_1608Metric_Pad0.98x0.95mm_HandSolder, F.Cu at (134.3, 128.5)
- added R9: 100k, Resistor_SMD:R_0603_1608Metric_Pad0.98x0.95mm_HandSolder, F.Cu at (138.6, 121.0)
- added SW2: RotaryEncoder_Switch, Rotary_Encoder:RotaryEncoder_Bourns_Vertical_PEC12R-3x17F-Sxxxx, F.Cu at (129.3, 109.4)
- added U3: AD8606ARZ, Package_SO:SOIC-8_3.9x4.9mm_P1.27mm, F.Cu at (145.0, 123.1)
- added U4: LMV331, Package_TO_SOT_SMD:SOT-23-5_HandSoldering, F.Cu at (148.3, 106.4)
- added U5: FSA3157L6X, Package_TO_SOT_SMD:SOT-363_SC-70-6, F.Cu at (147.5, 110.8)
- moved U2 40.1 mm to (57.8, 58.7)
Connections:
- U1 pad 2: unconnected-(U1-DGND-Pad2) -> GND
- U1 pad 6: unconnected-(U1-AGND-Pad6) -> GND

Commit message: Progress.
Parts:
- removed U4: LMV331, Package_TO_SOT_SMD:SOT-23-5_HandSoldering
- added C1: 100n, Capacitor_SMD:C_0603_1608Metric_Pad1.08x0.95mm_HandSolder, F.Cu at (116.7, 47.8)
- added C10: 47u, Capacitor_THT:CP_Radial_D5.0mm_P2.00mm, F.Cu at (100.1, 101.0)
- added C11: 47u, Capacitor_THT:CP_Radial_D5.0mm_P2.00mm, F.Cu at (100.1, 107.6)
- added C12: 47u, Capacitor_THT:CP_Radial_D5.0mm_P2.00mm, F.Cu at (106.8, 94.5)
- added C13: 47u, Capacitor_THT:CP_Radial_D5.0mm_P2.00mm, F.Cu at (106.8, 101.0)
- added C14: 1u, Resistor_SMD:R_0603_1608Metric_Pad0.98x0.95mm_HandSolder, F.Cu at (119.8, 115.6)
- added C15: 1u, Resistor_SMD:R_0603_1608Metric_Pad0.98x0.95mm_HandSolder, F.Cu at (119.8, 118.1)
- added C16: 47u, Capacitor_THT:CP_Radial_D5.0mm_P2.00mm, F.Cu at (106.8, 107.6)
- added C17: 1u, Resistor_SMD:R_0603_1608Metric_Pad0.98x0.95mm_HandSolder, F.Cu at (119.8, 120.6)
- added C18: 1u, Resistor_SMD:R_0603_1608Metric_Pad0.98x0.95mm_HandSolder, F.Cu at (119.8, 123.1)
- added C19: 1u, Resistor_SMD:R_0603_1608Metric_Pad0.98x0.95mm_HandSolder, F.Cu at (119.8, 125.6)
- added C2: 100n, Capacitor_SMD:C_0603_1608Metric_Pad1.08x0.95mm_HandSolder, F.Cu at (116.7, 50.3)
- added C20: 47u, Capacitor_THT:CP_Radial_D5.0mm_P2.00mm, F.Cu at (113.4, 94.5)
- added C21: 47u, Capacitor_THT:CP_Radial_D5.0mm_P2.00mm, F.Cu at (113.4, 101.0)
- added C22: 1u, Resistor_SMD:R_0603_1608Metric_Pad0.98x0.95mm_HandSolder, F.Cu at (124.2, 110.5)
- added C23: 1u, Resistor_SMD:R_0603_1608Metric_Pad0.98x0.95mm_HandSolder, F.Cu at (124.2, 113.0)
- added C24: 47u, Capacitor_THT:CP_Radial_D5.0mm_P2.00mm, F.Cu at (113.4, 107.6)
- added C4: 100n, Capacitor_SMD:C_0603_1608Metric_Pad1.08x0.95mm_HandSolder, F.Cu at (116.7, 52.8)
- added C5: 100n, Capacitor_SMD:C_0603_1608Metric_Pad1.08x0.95mm_HandSolder, F.Cu at (116.7, 55.3)
- added C7: 47u, Capacitor_THT:CP_Radial_D5.0mm_P2.00mm, F.Cu at (100.1, 94.5)
- added C8: 1u, Resistor_SMD:R_0603_1608Metric_Pad0.98x0.95mm_HandSolder, F.Cu at (119.8, 110.5)
- added C9: 1u, Resistor_SMD:R_0603_1608Metric_Pad0.98x0.95mm_HandSolder, F.Cu at (119.8, 113.0)
- added D1: SK16, Diode_SMD:D_SMA_Handsoldering, F.Cu at (131.8, 93.5)
- added J1: Conn_Coaxial, Connector_Coaxial:BNC_Amphenol_B6252HB-NPP3G-50_Horizontal, F.Cu at (106.1, 80.9)
- added L1: 4.7u, Inductor_THT:L_Radial_D7.5mm_P3.50mm_Fastron_07P, F.Cu at (120.4, 95.7)
- added L2: 4.7u, Inductor_THT:L_Radial_D7.5mm_P3.50mm_Fastron_07P, F.Cu at (120.4, 104.8)
- added Q1: J111, Package_TO_SOT_THT:TO-92, F.Cu at (135.6, 84.6)
- added Q2: MMBF4393, Package_TO_SOT_SMD:SOT-23, F.Cu at (107.6, 86.5)
- added Q5: BD679, Package_TO_SOT_THT:TO-126-3_Horizontal_TabUp, F.Cu at (100.3, 112.5)
- added Q6: BD680, Package_TO_SOT_THT:TO-126-3_Horizontal_TabUp, F.Cu at (109.8, 112.5)
- added R13: 1k, Resistor_SMD:R_0603_1608Metric_Pad0.98x0.95mm_HandSolder, F.Cu at (125.4, 47.8)
- added R14: 100k, Resistor_SMD:R_0603_1608Metric_Pad0.98x0.95mm_HandSolder, F.Cu at (125.4, 50.3)
- added R15: 1k, Resistor_SMD:R_0603_1608Metric_Pad0.98x0.95mm_HandSolder, F.Cu at (125.4, 52.8)
- added R16: 2.2k, Resistor_SMD:R_0603_1608Metric_Pad0.98x0.95mm_HandSolder, F.Cu at (125.4, 55.3)
- added R17: 1k, Resistor_SMD:R_0603_1608Metric_Pad0.98x0.95mm_HandSolder, F.Cu at (125.4, 57.9)
- added R18: 1k, Resistor_SMD:R_0603_1608Metric_Pad0.98x0.95mm_HandSolder, F.Cu at (125.4, 60.4)
- added R19: 1k, Resistor_SMD:R_0603_1608Metric_Pad0.98x0.95mm_HandSolder, F.Cu at (125.4, 62.9)
- added R20: 1k, Resistor_SMD:R_0603_1608Metric_Pad0.98x0.95mm_HandSolder, F.Cu at (125.4, 65.4)
- added R21: 5.1k, Resistor_SMD:R_0603_1608Metric_Pad0.98x0.95mm_HandSolder, F.Cu at (124.2, 115.6)
- added R22: 5.1k, Resistor_SMD:R_0603_1608Metric_Pad0.98x0.95mm_HandSolder, F.Cu at (124.2, 118.1)
- added R25: 2.2k, Resistor_SMD:R_0603_1608Metric_Pad0.98x0.95mm_HandSolder, F.Cu at (129.7, 47.8)
- added R26: 1k, Resistor_SMD:R_0603_1608Metric_Pad0.98x0.95mm_HandSolder, F.Cu at (129.7, 50.3)
- added R27: 2k, Resistor_SMD:R_0603_1608Metric_Pad0.98x0.95mm_HandSolder, F.Cu at (129.7, 52.8)
- added R28: 50, Resistor_SMD:R_0603_1608Metric_Pad0.98x0.95mm_HandSolder, F.Cu at (129.7, 55.3)
- added R29: 1k, Resistor_SMD:R_0603_1608Metric_Pad0.98x0.95mm_HandSolder, F.Cu at (124.2, 120.6)
- added R30: 1k, Resistor_SMD:R_0603_1608Metric_Pad0.98x0.95mm_HandSolder, F.Cu at (124.2, 123.1)
- added R31: 10k, Resistor_SMD:R_0603_1608Metric_Pad0.98x0.95mm_HandSolder, F.Cu at (124.2, 125.6)
- added R32: 10k, Resistor_SMD:R_0603_1608Metric_Pad0.98x0.95mm_HandSolder, F.Cu at (128.5, 110.5)
- added R33: 33k, Resistor_SMD:R_0603_1608Metric_Pad0.98x0.95mm_HandSolder, F.Cu at (128.5, 113.0)
- added R34: 33k, Resistor_SMD:R_0603_1608Metric_Pad0.98x0.95mm_HandSolder, F.Cu at (128.5, 115.6)
- added R35: 249.9k, Resistor_SMD:R_0603_1608Metric_Pad0.98x0.95mm_HandSolder, F.Cu at (128.5, 118.1)
- added RV1: 50k, Potentiometer_THT:Potentiometer_Bourns_3296W_Vertical, F.Cu at (137.5, 69.9)
- added U11: LM7171, Package_SO:SOIC-8_3.9x4.9mm_P1.27mm, F.Cu at (136.1, 63.1)
- added U13: LMR62421XMF, Package_TO_SOT_SMD:SOT-23-5, F.Cu at (133.3, 111.7)
- added U6: AD8039, Package_SO:SOIC-8_3.9x4.9mm_P1.27mm, F.Cu at (136.1, 56.5)
- added U7: LM393LVDDFR, Package_TO_SOT_SMD:SOT-223-8, F.Cu at (134.9, 77.2)
- added U8: FSA3157L6X, Package_TO_SOT_SMD:SOT-363_SC-70-6, F.Cu at (131.5, 83.3)
- added U9: FSA3157L6X, Package_TO_SOT_SMD:SOT-363_SC-70-6, F.Cu at (131.5, 87.3)
- R10: value 100k -> 100
- R11: value 1k -> 100
- R12: value 2k -> 100k
- R2: value 2k -> 10k
- R3: value 1k -> 20k
- R4, R8: value 2k -> 33k
- R5: value 100k -> 33k
- R6: value 100k -> 10k
- R7: value 1k -> 100k
- R9: value 100k -> 150k
- U3: value AD8606ARZ -> AD8039
- U5: value FSA3157L6X -> AD5258BRM; footprint Package_TO_SOT_SMD:SOT-363_SC-70-6 -> Package_SO:MSOP-10_3x3mm_P0.5mm
- moved R5 74.4 mm to (121.0, 47.8)
- moved R6 74.4 mm to (121.0, 50.3)
- moved R7 74.4 mm to (121.0, 52.8)
- moved R8 74.4 mm to (121.0, 55.3)
- moved U3 73.7 mm to (136.1, 49.9)
- moved R11 65.6 mm to (121.0, 62.9)
- moved R12 65.6 mm to (121.0, 65.4)
- moved R9 65.6 mm to (121.0, 57.9)
- moved R10 65.6 mm to (121.0, 60.4)
- moved SW2 64.8 mm to (79.7, 67.7)
- moved R1 64.5 mm to (116.7, 57.9)
- moved R3 64.5 mm to (116.7, 62.9)
- moved R4 64.5 mm to (116.7, 65.4)
- moved R2 64.5 mm to (116.7, 60.4)
- moved U5 52.1 mm to (101.5, 86.4)
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Connections:
- R1 pad 1: Net-(R1-Pad1) -> /AMP/GAIN_SET_DAC
- R1 pad 2: Net-(U3B-+) -> Net-(U4A-+)
- R10 pad 1: GND -> Net-(R10-Pad1)
- R11 pad 1: Net-(R11-Pad1) -> Net-(R10-Pad2)
- R11 pad 2: Net-(U3A--) -> Net-(Q1-D)
- R12 pad 1: Net-(U3A--) -> Net-(Q1-G)
- R12 pad 2: Net-(U4-+) -> Net-(R12-Pad2)
- R2 pad 1: Net-(U3B--) -> GND
- R2 pad 2: Net-(R2-Pad2) -> Net-(U6A--)
- R3 pad 1: Net-(R3-Pad1) -> GND
- R3 pad 2: Net-(U3B--) -> Net-(U4B-+)
- R4 pad 1: GND -> Net-(U4A--)
- R4 pad 2: Net-(U3B-+) -> Net-(U4B--)
- R5 pad 1: Net-(R5-Pad1) -> Net-(U4A--)
- R5 pad 2: +3V3 -> Net-(U4B--)
- R6 pad 1: GND -> Net-(U6A--)
- R7 pad 1: Net-(U1-OUT) -> Net-(U4B-+)
- R7 pad 2: Net-(U3A-+) -> +5V
- R8 pad 1: GND -> Net-(R6-Pad2)
- R8 pad 2: Net-(U3A-+) -> Net-(U7A--)
- R9 pad 1: Net-(R9-Pad1) -> OUT_3V3
- R9 pad 2: +3V3 -> Net-(R10-Pad1)
- U1 pad 1: unconnected-(U1-V_{cc}-Pad1) -> +5V
- U2 pad 18: unconnected-(U2-5V-Pad18) -> +VBUS
- U2 pad 19: unconnected-(U2-GND-Pad19) -> GND
- U2 pad 25: unconnected-(U2-PA0-Pad25) -> /AMP/GAIN_SET_DAC
- U2 pad 26: unconnected-(U2-PA1-Pad26) -> /AMP/SQUARE_SEL
- U2 pad 27: unconnected-(U2-PA2-Pad27) -> /AMP/PWM_SEL
- U2 pad 28: unconnected-(U2-PA3-Pad28) -> /AMP/DC_OFFSET_PWM
- U2 pad 29: unconnected-(U2-PA4-Pad29) -> /AMP/PWM_THRS_DAC
- U2 pad 39: unconnected-(U2-GND-Pad39) -> GND
- U2 pad 40: unconnected-(U2-GND-Pad40) -> GND
- U2 pad 41: unconnected-(U2-GND-Pad41) -> GND
- U3 pad 1: Net-(U4-+) -> OUT_3V3
- U3 pad 2: Net-(U3A--) -> OUT_3V3
- U3 pad 4: unconnected-(U3C-V--Pad4) -> -5V
- U3 pad 5: Net-(U3B-+) -> Net-(Q1-D)
- U3 pad 7: Net-(R2-Pad2) -> Net-(U3B--)
- U3 pad 8: unconnected-(U3C-V+-Pad8) -> +5V
- U5 pad 1: Net-(U4-Pad4) -> Net-(Q1-D)
- U5 pad 2: (no net) -> unconnected-(U5-AD0-Pad2)
- U5 pad 3: Net-(U4-+) -> unconnected-(U5-AD1-Pad3)
- U5 pad 4: Net-(R1-Pad1) -> unconnected-(U5-SDA-Pad4)
- U5 pad 5: (no net) -> unconnected-(U5-SCL-Pad5)

Commit message: Savegame.
Parts:
- removed C1, C2: 100n, Capacitor_SMD:C_0603_1608Metric_Pad1.08x0.95mm_HandSolder
- added C25: 100n, Capacitor_SMD:C_0603_1608Metric_Pad1.08x0.95mm_HandSolder, F.Cu at (146.2, 86.5)
- added C26: 1u, Resistor_SMD:R_0603_1608Metric_Pad0.98x0.95mm_HandSolder, F.Cu at (132.1, 76.4)
- added C27: 1u, Resistor_SMD:R_0603_1608Metric_Pad0.98x0.95mm_HandSolder, F.Cu at (116.0, 69.3)
- added C28: 1u, Resistor_SMD:R_0603_1608Metric_Pad0.98x0.95mm_HandSolder, F.Cu at (109.3, 82.4)
- added C29: 100n, Resistor_SMD:R_0603_1608Metric_Pad0.98x0.95mm_HandSolder, F.Cu at (116.0, 70.8)
- added C3: 1u, Resistor_SMD:R_0603_1608Metric_Pad0.98x0.95mm_HandSolder, F.Cu at (136.1, 66.4)
- added C30: 100n, Resistor_SMD:R_0603_1608Metric_Pad0.98x0.95mm_HandSolder, F.Cu at (109.3, 80.9)
- added C31: 1n, Resistor_SMD:R_0603_1608Metric_Pad0.98x0.95mm_HandSolder, F.Cu at (116.0, 72.3)
- added C32: 1n, Resistor_SMD:R_0603_1608Metric_Pad0.98x0.95mm_HandSolder, F.Cu at (109.3, 79.4)
- added C33: 1u, Resistor_SMD:R_0603_1608Metric_Pad0.98x0.95mm_HandSolder, F.Cu at (99.7, 97.3)
- added C34: 100n, Capacitor_SMD:C_0603_1608Metric_Pad1.08x0.95mm_HandSolder, F.Cu at (98.8, 77.0)
- added C35: 100n, Capacitor_SMD:C_0603_1608Metric_Pad1.08x0.95mm_HandSolder, F.Cu at (102.2, 96.6)
- added C36: 1u, Resistor_SMD:R_0603_1608Metric_Pad0.98x0.95mm_HandSolder, F.Cu at (160.1, 129.9)
- added C37: 1u, Resistor_SMD:R_0603_1608Metric_Pad0.98x0.95mm_HandSolder, F.Cu at (156.7, 127.5)
- added C38: 22p, Capacitor_SMD:C_0603_1608Metric_Pad1.08x0.95mm_HandSolder, F.Cu at (98.2, 84.3)
- added C39: 22p, Capacitor_SMD:C_0603_1608Metric_Pad1.08x0.95mm_HandSolder, F.Cu at (103.0, 84.4)
- added C40: 22p, Capacitor_SMD:C_0603_1608Metric_Pad1.08x0.95mm_HandSolder, F.Cu at (106.2, 84.3)
- added C41: 33p, Capacitor_SMD:C_0603_1608Metric_Pad1.08x0.95mm_HandSolder, F.Cu at (101.3, 84.4)
- added C42: 1p, Capacitor_SMD:C_0603_1608Metric_Pad1.08x0.95mm_HandSolder, F.Cu at (98.8, 80.1)
- added C43: 5.6p, Capacitor_SMD:C_0603_1608Metric_Pad1.08x0.95mm_HandSolder, F.Cu at (102.2, 80.1)
- added C44: 4.7p, Capacitor_SMD:C_0603_1608Metric_Pad1.08x0.95mm_HandSolder, F.Cu at (105.5, 80.1)
- added C45: 10n, Resistor_SMD:R_0603_1608Metric_Pad0.98x0.95mm_HandSolder, F.Cu at (152.0, 101.7)
- added C46: 10n, Resistor_SMD:R_0603_1608Metric_Pad0.98x0.95mm_HandSolder, F.Cu at (148.7, 101.7)
- added C47: 10n, Resistor_SMD:R_0603_1608Metric_Pad0.98x0.95mm_HandSolder, F.Cu at (145.4, 101.7)
- added C48: 10n, Resistor_SMD:R_0603_1608Metric_Pad0.98x0.95mm_HandSolder, F.Cu at (161.9, 101.7)
- added C49: 10n, Resistor_SMD:R_0603_1608Metric_Pad0.98x0.95mm_HandSolder, F.Cu at (158.6, 101.7)
- added C50: 10n, Resistor_SMD:R_0603_1608Metric_Pad0.98x0.95mm_HandSolder, F.Cu at (155.3, 101.7)
- added C51: 100n, Capacitor_SMD:C_0603_1608Metric_Pad1.08x0.95mm_HandSolder, F.Cu at (149.3, 67.8)
- added C52: 2.2u, Capacitor_SMD:C_1206_3216Metric_Pad1.33x1.80mm_HandSolder, F.Cu at (148.4, 65.9)
- added C53: 100n, Capacitor_SMD:C_0603_1608Metric_Pad1.08x0.95mm_HandSolder, F.Cu at (141.9, 75.1)
- added C54: 2.2u, Capacitor_SMD:C_1206_3216Metric_Pad1.33x1.80mm_HandSolder, F.Cu at (142.8, 77.0)
- added C55: 10n, Capacitor_SMD:C_0603_1608Metric_Pad1.08x0.95mm_HandSolder, F.Cu at (149.3, 69.3)
- added C56: 10n, Capacitor_SMD:C_0603_1608Metric_Pad1.08x0.95mm_HandSolder, F.Cu at (141.9, 73.6)
- added C57: 100n, Capacitor_SMD:C_0603_1608Metric_Pad1.08x0.95mm_HandSolder, F.Cu at (130.1, 96.3)
- added C58: 100n, Capacitor_SMD:C_0603_1608Metric_Pad1.08x0.95mm_HandSolder, F.Cu at (131.9, 96.3)
- added C59: 100n, Resistor_SMD:R_0603_1608Metric_Pad0.98x0.95mm_HandSolder, F.Cu at (136.1, 67.9)
- added C6: 100n, Capacitor_SMD:C_0603_1608Metric_Pad1.08x0.95mm_HandSolder, F.Cu at (146.2, 89.9)
- added C60: 100n, Resistor_SMD:R_0603_1608Metric_Pad0.98x0.95mm_HandSolder, F.Cu at (132.1, 74.9)
- added C61: 100n, Capacitor_SMD:C_0603_1608Metric_Pad1.08x0.95mm_HandSolder, F.Cu at (148.8, 78.3)
- added C62: 100n, Capacitor_SMD:C_0603_1608Metric_Pad1.08x0.95mm_HandSolder, F.Cu at (141.3, 85.0)
- added C63: 100n, Capacitor_SMD:C_0603_1608Metric_Pad1.08x0.95mm_HandSolder, F.Cu at (127.0, 86.9)
- added C64: 100n, Capacitor_SMD:C_0603_1608Metric_Pad1.08x0.95mm_HandSolder, F.Cu at (134.3, 93.9)
- added C65: 100n, Capacitor_SMD:C_0603_1608Metric_Pad1.08x0.95mm_HandSolder, B.Cu at (107.0, 70.6)
- added C66: 100n, Capacitor_SMD:C_0603_1608Metric_Pad1.08x0.95mm_HandSolder, B.Cu at (112.0, 71.2)
- added C67: 100n, Capacitor_SMD:C_0603_1608Metric_Pad1.08x0.95mm_HandSolder, F.Cu at (151.4, 85.2)
- added C68: 100n, Capacitor_SMD:C_0603_1608Metric_Pad1.08x0.95mm_HandSolder, F.Cu at (151.4, 83.4)
- added FB1: FerriteBead, Inductor_SMD:L_0603_1608Metric_Pad1.05x0.95mm_HandSolder, F.Cu at (102.2, 98.2)
- added FB2: FerriteBead, Inductor_SMD:L_0603_1608Metric_Pad1.05x0.95mm_HandSolder, F.Cu at (98.8, 78.5)
- added J2: USB_C_Receptacle_PowerOnly_6P, Connector_USB:USB_C_Receptacle_GCT_USB4125-xx-x_6P_TopMnt_Horizontal, F.Cu at (85.8, 139.3)
- added J3: Conn_01x02_Pin, Connector_PinHeader_2.54mm:PinHeader_1x02_P2.54mm_Vertical, F.Cu at (154.0, 130.3)
- added J4: Conn_01x03_Pin, Connector_PinHeader_2.54mm:PinHeader_1x03_P2.54mm_Vertical, F.Cu at (129.7, 58.3)
- added J5: Conn_01x04_Pin, Connector_PinHeader_2.54mm:PinHeader_1x04_P2.54mm_Vertical, F.Cu at (116.3, 100.3)
- added J6: Conn_01x03_Pin, Connector_PinHeader_2.54mm:PinHeader_1x03_P2.54mm_Vertical, F.Cu at (125.9, 58.3)
- added L3: 470n, Inductor_SMD:L_0603_1608Metric, F.Cu at (98.8, 81.8)
- added L4: 390n, Inductor_SMD:L_0603_1608Metric, F.Cu at (102.2, 81.8)
- added L5: 390n, Inductor_SMD:L_0603_1608Metric, F.Cu at (105.5, 81.8)
- added R23: 100k, Resistor_SMD:R_0603_1608Metric_Pad0.98x0.95mm_HandSolder, F.Cu at (143.8, 87.4)
- added R24: 1k, Resistor_SMD:R_0603_1608Metric_Pad0.98x0.95mm_HandSolder, F.Cu at (130.9, 93.9)
- added R36: 10k, Resistor_SMD:R_0603_1608Metric_Pad0.98x0.95mm_HandSolder, F.Cu at (148.7, 96.9)
- added R37: 10k, Resistor_SMD:R_0603_1608Metric_Pad0.98x0.95mm_HandSolder, F.Cu at (149.6, 99.3)
- added R38: 10k, Resistor_SMD:R_0603_1608Metric_Pad0.98x0.95mm_HandSolder, F.Cu at (152.0, 96.9)
- added R39: 10k, Resistor_SMD:R_0603_1608Metric_Pad0.98x0.95mm_HandSolder, F.Cu at (152.9, 99.3)
- added R40: 10k, Resistor_SMD:R_0603_1608Metric_Pad0.98x0.95mm_HandSolder, F.Cu at (145.4, 96.9)
- added R41: 10k, Resistor_SMD:R_0603_1608Metric_Pad0.98x0.95mm_HandSolder, F.Cu at (146.3, 99.3)
- added R42: 10k, Resistor_SMD:R_0603_1608Metric_Pad0.98x0.95mm_HandSolder, F.Cu at (161.9, 96.9)
- added R43: 10k, Resistor_SMD:R_0603_1608Metric_Pad0.98x0.95mm_HandSolder, F.Cu at (162.8, 99.3)
- added R44: 10k, Resistor_SMD:R_0603_1608Metric_Pad0.98x0.95mm_HandSolder, F.Cu at (158.6, 96.9)
- added R45: 10k, Resistor_SMD:R_0603_1608Metric_Pad0.98x0.95mm_HandSolder, F.Cu at (159.5, 99.3)
- added R46: 10k, Resistor_SMD:R_0603_1608Metric_Pad0.98x0.95mm_HandSolder, F.Cu at (155.3, 96.9)
- added R47: 10k, Resistor_SMD:R_0603_1608Metric_Pad0.98x0.95mm_HandSolder, F.Cu at (156.2, 99.3)
- added R48: 50, Resistor_SMD:R_0603_1608Metric_Pad0.98x0.95mm_HandSolder, F.Cu at (149.3, 72.3)
- added R49: 1k, Resistor_SMD:R_0603_1608Metric_Pad0.98x0.95mm_HandSolder, F.Cu at (148.9, 87.7)
- added R50: 1k, Resistor_SMD:R_0603_1608Metric_Pad0.98x0.95mm_HandSolder, F.Cu at (148.9, 84.3)
- added U10: TL072, Package_SO:SOIC-8_3.9x4.9mm_P1.27mm, F.Cu at (144.3, 81.4)
- added U12: L7805, Package_TO_SOT_THT:TO-220-3_Vertical, F.Cu at (125.2, 135.4)
- added U14: AP2204K-3.3, Package_TO_SOT_SMD:SOT-23-5, F.Cu at (159.7, 127.4)
- added U15: L7905, Package_TO_SOT_THT:TO-220-3_Vertical, F.Cu at (136.5, 135.4)
- added U16: Screen to I2C, PSG:screen_to_i2c, F.Cu at (166.0, 152.9)
- added U17: Screen, PSG:20x4 screen, F.Cu at (171.6, 132.4)
- added U4: TL072, Package_SO:SOIC-8_3.9x4.9mm_P1.27mm, F.Cu at (131.4, 89.4)
- Q1: footprint Package_TO_SOT_THT:TO-92 -> Package_TO_SOT_THT:TO-92_Inline_Wide
- Q5, Q6: footprint Package_TO_SOT_THT:TO-126-3_Horizontal_TabUp -> Package_TO_SOT_THT:TO-126-3_Vertical
- R17: value 1k -> 100k
- SW1, SW2: footprint Rotary_Encoder:RotaryEncoder_Bourns_Vertical_PEC12R-3x17F-Sxxxx -> PSG:RotaryEncoder_Bourns_Vertical_PEC12R-3x17F-Sxxxx
- U8, U9: footprint Package_TO_SOT_SMD:SOT-363_SC-70-6 -> Package_TO_SOT_SMD:SOT-23-6_Handsoldering
- moved U2 115.6 mm to (159.1, 106.5), turned to -90 degrees
- moved SW1 85.0 mm to (35.6, 124.6), turned to -90 degrees
- moved C7 59.8 mm to (137.2, 141.4)
- moved D1 50.7 mm to (111.1, 139.8), turned to 180 degrees
- moved C12 50.3 mm to (124.9, 141.4)
- moved J1 48.5 mm to (153.7, 71.3), turned to -90 degrees
- moved C4 48.2 mm to (98.0, 97.3), turned to 90 degrees
- moved L1 47.9 mm to (98.0, 138.1), turned to -90 degrees
- moved C11 47.6 mm to (133.5, 141.5), turned to 180 degrees
- moved SW2 45.3 mm to (43.9, 95.5), turned to -90 degrees
- moved C10 44.7 mm to (119.2, 141.4)
- moved L2 44.3 mm to (102.5, 145.2)
- moved U1 42.5 mm to (95.4, 98.4), turned to 180 degrees
- moved R5 42.0 mm to (126.4, 89.5), turned to 90 degrees
- moved C8 42.0 mm to (136.3, 149.2)
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Connections:
- C10 pad 2: 0 -> GND
- C11 pad 1: 0 -> GND
- C12 pad 2: 0 -> GND
- C13 pad 2: 0 -> GND
- C14 pad 2: 0 -> GND
- C15 pad 2: 0 -> GND
- C16 pad 2: 0 -> GND
- C17 pad 2: 0 -> GND
- C18 pad 2: 0 -> GND
- C19 pad 2: 0 -> GND
- C20 pad 2: 0 -> GND
- C21 pad 1: 0 -> GND
- C22 pad 2: 0 -> GND
- C23 pad 2: 0 -> GND
- C24 pad 1: 0 -> GND
- C4 pad 1: +5V -> Net-(U1-V_{cc})
- C5 pad 1: +3V3 -> +5V
- C7 pad 1: 0 -> GND
- C8 pad 2: 0 -> GND
- C9 pad 2: 0 -> GND
- R13 pad 2: +5V -> Net-(C34-Pad1)
- R15 pad 1: Net-(U3B--) -> Net-(U6A--)
- R2 pad 2: Net-(U6A--) -> Net-(U3A--)
- R31 pad 1: 0 -> GND
- R32 pad 1: 0 -> GND
- R6 pad 1: Net-(U6A--) -> Net-(U3A--)
- SW1 pad A: unconnected-(SW1-PadA) -> Net-(R38-Pad1)
- SW1 pad B: unconnected-(SW1-PadB) -> Net-(R36-Pad1)
- SW1 pad C: unconnected-(SW1-PadC) -> GND
- SW1 pad S1: unconnected-(SW1-PadS1) -> Net-(R40-Pad1)
- SW1 pad S2: unconnected-(SW1-PadS2) -> GND
- SW2 pad A: unconnected-(SW2-PadA) -> Net-(R42-Pad1)
- SW2 pad B: unconnected-(SW2-PadB) -> Net-(R44-Pad1)
- SW2 pad C: unconnected-(SW2-PadC) -> GND
- SW2 pad S1: unconnected-(SW2-PadS1) -> Net-(R46-Pad1)
- SW2 pad S2: unconnected-(SW2-PadS2) -> GND
- U1 pad 1: +5V -> Net-(U1-V_{cc})
- U1 pad 3: unconnected-(U1-SDATA-Pad3) -> /AMP/SDATA_SG
- U1 pad 4: unconnected-(U1-SCLK-Pad4) -> /AMP/SCK_SG
- U1 pad 5: unconnected-(U1-FSYNC-Pad5) -> /AMP/FSYNC_SG
- U2 pad 1: unconnected-(U2-PB12-Pad1) -> EN_A_2
- U2 pad 14: unconnected-(U2-PB6-Pad14) -> SCL_1
- U2 pad 15: unconnected-(U2-PB7-Pad15) -> SDA_1
- U2 pad 16: unconnected-(U2-PB8-Pad16) -> /MCU/SDA_2
- U2 pad 17: unconnected-(U2-PB9-Pad17) -> /MCU/SCL_2
- U2 pad 2: unconnected-(U2-PB13-Pad2) -> EN_B_2
- U2 pad 20: unconnected-(U2-3V3-Pad20) -> +3.3V_MCU
- U2 pad 22: unconnected-(U2-PC13-Pad22) -> /AMP/SQUARE_SEL
- U2 pad 23: unconnected-(U2-PC14-Pad23) -> /AMP/PWM_SEL
- U2 pad 26: /AMP/SQUARE_SEL -> /AMP/DC_OFFSET_PWM
- U2 pad 27: /AMP/PWM_SEL -> /AMP/PWM_THRS_DAC
- U2 pad 28: /AMP/DC_OFFSET_PWM -> unconnected-(U2-PA3-Pad28)
- U2 pad 29: /AMP/PWM_THRS_DAC -> unconnected-(U2-PA4-Pad29)
- U2 pad 3: unconnected-(U2-PB14-Pad3) -> EN_SW_2
- U2 pad 30: unconnected-(U2-PA5-Pad30) -> /AMP/SDATA_SG
- U2 pad 32: unconnected-(U2-PA7-Pad32) -> /AMP/SCK_SG
- U2 pad 33: unconnected-(U2-PB0-Pad33) -> /AMP/FSYNC_SG
- U2 pad 38: unconnected-(U2-3V3-Pad38) -> +3.3V_MCU
- U2 pad 4: unconnected-(U2-PB15-Pad4) -> EN_A_1
- U2 pad 44: unconnected-(U2-3V3-Pad44) -> +3.3V_MCU
- U2 pad 5: unconnected-(U2-PA8-Pad5) -> EN_B_1
- U2 pad 6: unconnected-(U2-PA9-Pad6) -> EN_SW_1
- U3 pad 1: OUT_3V3 -> Net-(U7A--)
- U3 pad 2: OUT_3V3 -> Net-(U3A--)
- U3 pad 5: Net-(Q1-D) -> Net-(U3B-+)
- U3 pad 6: Net-(U3B--) -> OUT_3V3
- U3 pad 7: Net-(U3B--) -> OUT_3V3
- U5 pad 2: unconnected-(U5-AD0-Pad2) -> Net-(J6-Pin_2)
- U5 pad 3: unconnected-(U5-AD1-Pad3) -> Net-(J4-Pin_2)
- U5 pad 4: unconnected-(U5-SDA-Pad4) -> /AMP/SDA_2
- U5 pad 5: unconnected-(U5-SCL-Pad5) -> /AMP/SCL_2
- U5 pad 6: unconnected-(U5-V_{LOGIC}-Pad6) -> +3.3V
- U5 pad 8: unconnected-(U5-VDD-Pad8) -> +5V
- U6 pad 1: Net-(U7A--) -> Net-(U6A--)
- U6 pad 3: Net-(U1-OUT) -> Net-(Q1-D)
- U7 pad 3: /AMP/PWM_THRS_DAC -> Net-(U10B--)
- U7 pad 5: unconnected-(U7B-+-Pad5) -> +5V
- U7 pad 6: unconnected-(U7B---Pad6) -> GND
- U8 pad 2: (no net) -> GND
- U8 pad 5: (no net) -> +5V
- U9 pad 2: (no net) -> GND
- U9 pad 3: Net-(U1-OUT) -> Net-(U3A-+)
- U9 pad 4: Net-(U3A-+) -> Net-(U3B-+)
- U9 pad 5: (no net) -> +5V
Other:
- board outline added: 80.8 x 100 mm

Commit message: Added readme.
Parts:
- added J10: Conn_01x01_Pin, Connector_PinHeader_2.54mm:PinHeader_1x01_P2.54mm_Vertical, F.Cu at (147.4, 94.2)
- added J11: Conn_01x01_Pin, Connector_PinHeader_2.54mm:PinHeader_1x01_P2.54mm_Vertical, F.Cu at (158.2, 90.5)
- added J12: Conn_01x01_Pin, Connector_PinHeader_2.54mm:PinHeader_1x01_P2.54mm_Vertical, F.Cu at (161.8, 94.2)
- added J13: Conn_01x01_Pin, Connector_PinHeader_2.54mm:PinHeader_1x01_P2.54mm_Vertical, F.Cu at (161.8, 90.5)
- added J14: Conn_01x01_Pin, Connector_PinHeader_2.54mm:PinHeader_1x01_P2.54mm_Vertical, F.Cu at (158.2, 94.2)
- added J15: Conn_01x01_Pin, Connector_PinHeader_2.54mm:PinHeader_1x01_P2.54mm_Vertical, F.Cu at (154.6, 94.2)
- added J16: Conn_01x01_Pin, Connector_PinHeader_2.54mm:PinHeader_1x01_P2.54mm_Vertical, F.Cu at (154.6, 90.5)
- added J7: Conn_01x01_Pin, Connector_PinHeader_2.54mm:PinHeader_1x01_P2.54mm_Vertical, F.Cu at (151.0, 94.2)
- added J8: Conn_01x01_Pin, Connector_PinHeader_2.54mm:PinHeader_1x01_P2.54mm_Vertical, F.Cu at (151.0, 90.5)
- added J9: Conn_01x01_Pin, Connector_PinHeader_2.54mm:PinHeader_1x01_P2.54mm_Vertical, F.Cu at (140.0, 100.2)
- moved SW1 148.0 mm to (160.8, 45.5), turned to 0 degrees
- moved SW2 119.9 mm to (160.8, 68.5), turned to 0 degrees
- moved R49 1.38 mm to (149.9, 86.7), turned to 180 degrees
- moved U16 0.89 mm to (166.9, 153.0)
Connections:
- R36 pad 1: Net-(R36-Pad1) -> Net-(J9-Pin_1)
- R37 pad 2: Net-(R36-Pad1) -> Net-(J9-Pin_1)
- R38 pad 1: Net-(R38-Pad1) -> Net-(J7-Pin_1)
- R39 pad 2: Net-(R38-Pad1) -> Net-(J7-Pin_1)
- R40 pad 1: Net-(R40-Pad1) -> Net-(J10-Pin_1)
- R41 pad 2: Net-(R40-Pad1) -> Net-(J10-Pin_1)
- R42 pad 1: Net-(R42-Pad1) -> Net-(J12-Pin_1)
- R43 pad 2: Net-(R42-Pad1) -> Net-(J12-Pin_1)
- R44 pad 1: Net-(R44-Pad1) -> Net-(J14-Pin_1)
- R45 pad 2: Net-(R44-Pad1) -> Net-(J14-Pin_1)
- R46 pad 1: Net-(R46-Pad1) -> Net-(J15-Pin_1)
- R47 pad 2: Net-(R46-Pad1) -> Net-(J15-Pin_1)
Other:
- board size 80.8 x 100 mm -> 80.8 x 96.1 mm
