File: _autosave-mcu.kicad_sch (KiCad schematic)
At the start: 35 parts, among them J10 Conn_01x01_Pin, J11 Conn_01x01_Pin, J12 Conn_01x01_Pin, J13 Conn_01x01_Pin, J14 Conn_01x01_Pin, J15 Conn_01x01_Pin, J16 Conn_01x01_Pin, J3 Conn_01x02_Pin, J5 Conn_01x04_Pin, J7 Conn_01x01_Pin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

Commit message: Added readme.
Other:
- moved on the sheet: SW1, SW2
Changed lines of the file:
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@@
 		(lib_name "RotaryEncoder_Switch_1")
 		(lib_id "PSG:RotaryEncoder_Switch")
-		(at 125.73 116.84 0)
-		(unit 1)
-		(exclude_from_sim no)
-		(in_bom yes)
-		(on_board yes)
-		(dnp no)
-		(fields_autoplaced yes)
+		(at 137.16 147.32 0)
+		(unit 1)
+		(exclude_from_sim no)
+		(in_bom yes)
+		(on_board yes)
+		(dnp no)
 		(property "Reference" "SW2"
-			(at 125.73 106.68 0)
+			(at 136.906 139.954 0)
 			(effects
 				(font
@@
 		)
 		(property "Value" "RotaryEncoder_Switch"
-			(at 125.73 109.22 0)
-			(effects
-				(font
-					(size 1.27 1.27)
-				)
+			(at 137.16 139.7 0)
+			(effects
+				(font
+					(size 1.27 1.27)
+				)
+				(hide yes)
 			)
 		)
 		(property "Footprint" "PSG:RotaryEncoder_Bourns_Vertical_PEC12R-3x17F-Sxxxx"
-			(at 121.92 112.776 0)
+			(at 133.35 143.256 0)
 			(effects
 				(font
@@
 		)
 		(property "Datasheet" "~"
-			(at 125.73 110.236 0)
+			(at 137.16 140.716 0)
 			(effects
 				(font
@@
 		)
 		(property "Description" "Rotary encoder, dual channel, incremental quadrate outputs, with switch"
-			(at 125.73 116.84 0)
+			(at 137.16 147.32 0)
 			(effects
 				(font
@@
 	(symbol
 		(lib_id "PSG:RotaryEncoder_Switch")
-		(at 43.18 116.84 0)
-		(unit 1)
-		(exclude_from_sim no)
-		(in_bom yes)
-		(on_board yes)
-		(dnp no)
-		(fields_autoplaced yes)
+		(at 53.34 147.32 0)
+		(unit 1)
+		(exclude_from_sim no)
+		(in_bom yes)
+		(on_board yes)
+		(dnp no)
 		(property "Reference" "SW1"
-			(at 43.18 106.68 0)
+			(at 53.086 140.716 0)
 			(effects
 				(font
@@
 		)
 		(property "Value" "RotaryEncoder_Switch"
-			(at 43.18 109.22 0)
-			(effects
-				(font
-					(size 1.27 1.27)
-				)
+			(at 53.34 139.7 0)
+			(effects
+				(font
+					(size 1.27 1.27)
+				)
+				(hide yes)
 			)
 		)
 		(property "Footprint" "PSG:RotaryEncoder_Bourns_Vertical_PEC12R-3x17F-Sxxxx"
-			(at 39.37 112.776 0)
+			(at 49.53 143.256 0)
 			(effects
 				(font
@@
 		)
 		(property "Datasheet" "~"
-			(at 43.18 110.236 0)
+			(at 53.34 140.716 0)
 			(effects
 				(font
@@
 		)
 		(property "Description" "Rotary encoder, dual channel, incremental quadrate outputs, with switch"
-			(at 43.18 116.84 0)
-			(effects
-				(font
+			(at 53.34 147.32 0)
+			(effects
+				(font
